Commit message: four bar linkage

File: mengine/assets/fourbarlinkage.urdf (robot description, URDF)
Before this commit: robot simple_arm, 6 links, 5 joints
Links:
- added link link_ee
- link link3: geometry visual capsule length=0.1 radius=0.02
Joints:
- added joint joint_ee: type revolute, parent link4, child link_ee, origin xyz=0 -0.4 0 rpy=0 0 0, axis 1 0 0, limit effort=100 velocity=10
- joint joint3: origin xyz=0 0 0.2 rpy=0 0 0 -> xyz=0 0 0.1 rpy=0 0 0

Commit message: add inertial properties to all links (stops the b3prints complaining about not having this data)

File: mengine/assets/fourbarlinkage.urdf (robot description, URDF)
Before this commit: robot simple_arm, 7 links, 6 joints
Links:
- link base_link: mass None -> 1
- link link2: mass None -> 1
- link link3: mass None -> 1
- link link4: mass None -> 1
- link link5: mass None -> 1
- link link6: mass None -> 1
- link link_ee: mass None -> 1
