Commit message: Stretch 3

File: mengine/assets/stretch3/stretch_description_SE3_eoa_wrist_dw3_tool_sg3.urdf (robot description, URDF)
Before this commit: robot stretch, 61 links, 60 joints
Joints:
- joint joint_gripper_finger_left: limit lower=0 upper=0 effort=0 velocity=0 -> lower=0 upper=0.5 effort=0 velocity=0
- joint joint_gripper_finger_right: limit lower=0 upper=0 effort=0 velocity=0 -> lower=0 upper=0.5 effort=0 velocity=0
